File: kikad/platy/platy.kicad_sch (KiCad schematic)
At the start: 108 parts, among them J1 Conn_01x10, J2 Conn_01x08, J3 USB_C_Receptacle_USB2.0_16P, Q1 2N7002, Q2 2N7002, SW1 SW_DPST, U1 ESP32-S3, U2 APS6404L-3SQRx-SN, U3 W25Q128JVS, U4 CC1101, U5 PN5321A3HN_C1xx, U6 AMS1117-3.3, U7 ESP32-S3-WROOM-1, Y1 40Mhz(+-10 ppm), Y2 Crystal, Y3 27.12Mhz

Commit message: added the microsd card and the made changes in the schiematic
Parts:
- removed C? (x2): 0.1uF, symbol Device:C
- removed C?: 470pF, symbol Device:C
- removed C?: 10pF, symbol Device:C
- removed D?: BPW34, OptoDevice:Osram_DIL2_4.3x4.65mm_P5.08mm, symbol Sensor_Optical:BPW34
- removed D?: LED, symbol Device:LED
- removed Q?: Q_NPN, symbol Device:Q_NPN
- removed R? (x3): 10k, symbol Device:R
- removed R?: 220 ohm, symbol Device:R
- removed R? (x2): 100 ohm, symbol Device:R
- removed R? (x2): 100k, symbol Device:R
- removed SW?: SW_Push(Boot), symbol Switch:SW_Push
- removed SW?: SW_Push(EN), symbol Switch:SW_Push
- removed U? (x3): TLV9062, symbol Amplifier_Operational:TLV9062
- removed U? (x2): LM393, symbol Comparator:LM393
- added C33: 10pF, symbol Device:C
- added C34: 470pF, symbol Device:C
- added C35, C36: 0.1uF, symbol Device:C
- added C37: 100nF, symbol Device:C_Small
- added C38, C41, C42: 100nF, symbol Device:C
- added C39, C40, C43: 220nF, symbol Device:C
- added D10, D11: 1N5822, Diode_THT:D_DO-201AD_P15.24mm_Horizontal, symbol Diode:1N5822
- added D6: BPW34, OptoDevice:Osram_DIL2_4.3x4.65mm_P5.08mm, symbol Sensor_Optical:BPW34
- added D7: LED, symbol Device:LED
- added D8: IR led, symbol Device:LED
- added D9: D_TVS, symbol Device:D_TVS
- added F1: Fuse, symbol Device:Fuse
- added J4: Conn_01x02_Socket, symbol Connector:Conn_01x02_Socket
- added L5, L6: 33uH, symbol Device:L
- added Q3: Q_NPN, symbol Device:Q_NPN
- added Q4: BC847, Package_TO_SOT_SMD:SOT-23, symbol Transistor_BJT:BC847
- added Q5: Q_PMOS_GSD, symbol Transistor_FET:Q_PMOS_GSD
- added R26: 220 ohm, symbol Device:R
- added R27, R29: 100 ohm, symbol Device:R
- added R28, R30, R37: 100k, symbol Device:R
- added R31, R32, R33: 10k, symbol Device:R
- added R34: R_Small, symbol Device:R_Small
- added R35: 100, symbol Device:R
- added R36: 1K, symbol Device:R
- added R38: 1.68k, symbol Device:R
- added R39: 1k, symbol Device:R
- added SW2: SW_Push(Boot), symbol Switch:SW_Push
- added SW3: SW_Push(EN), symbol Switch:SW_Push
- added U10: TSOP382xx, OptoDevice:Vishay_MINICAST-3Pin, symbol Interface_Optical:TSOP382xx
- added U11: LM2596S-5, Package_TO_SOT_SMD:TO-263-5_TabPin3, symbol Regulator_Switching:LM2596S-5
- added U12: LM2596S-3.3, Package_TO_SOT_SMD:TO-263-5_TabPin3, symbol Regulator_Switching:LM2596S-3.3
- added U8: TLV9062, symbol Amplifier_Operational:TLV9062
- added U9: LM393, symbol Comparator:LM393
Connections:
- net +3V3: now also C42.1, C43.1, D6.1 (K), L6.2, R29.2, R31.1, R32.1, R33.1, R34.2, R35.1, R38.2, U8.8 (V+), U9.8 (V+)
- net +5V: now also C40.1, C41.1, L5.2, U11.4 (FB)
- net BOOT: now also C35.1, R32.2, SW2.1, SW2.2
- net EN: now also C36.1, R33.2, SW3.1, SW3.2
- net GND: now also C35.2, C36.2, C37.2, C38.2, C39.2, C40.2, C41.2, C42.2, C43.2, D10.2 (A), D11.2 (A), D9.2 (A2), Q3.E, Q4.2 (E), R27.2, R37.2, R39.2, U10.2 (GND), U11.3 (GND), U11.5 (~{ON}/OFF), U12.3 (GND), U12.5 (~{ON}/OFF), U8.3 (+), U8.4 (V-), U8.5 (+), U9.2 (-), U9.4 (V-)
- net IN: now also R26.1
- net OUT: now also R31.2, U9.1
- net GPIO 4: now reaches U7.4 (IO4)
- net GPIO 4: now also C37.1, U10.1 (OUT)
- net gpio 6: now reaches U7.6 (IO6)
- net gpio 6: now also R36.2
- new net: D8.1 (K), Q4.3 (C)
- new net: D8.2 (A), R35.2
- new net: C33.2, C34.1, R28.2, U8.1
- new net: C34.2, R30.1, U8.6 (-)
- new net: R30.2, U8.7, U9.3 (+)
- new net: D7.1 (K), Q3.C
- new net: D7.2 (A), R29.1
- new net: Q3.B, R26.2, R27.1
- new net: R34.1, U10.3 (Vs)
- new net: Q4.1 (B), R36.1
- new net: D10.1 (K), L5.1, U11.2 (OUT)
- new net: D11.1 (K), L6.1, U12.2 (OUT)
- new net: R38.1, R39.1, U12.4 (FB)
- new net: C33.1, D6.2 (A), R28.1, U8.2 (-)
- new net: F1.2, Q5.3 (D)
- new net: Q5.1 (G), R37.1
- new net BAT+: F1.1, J4.1 (Pin_1)
- new net Gnd: J4.2 (Pin_2)
- new net Vin: C38.1, C39.1, D9.1 (A1), Q5.2 (S), U11.1 (VIN), U12.1 (VIN)
Other:
- note added: "Battery"
- note added: "IR Transmitter"
- note added: "IR receiver"
- moved on the sheet: C1, C10, C11, C12, C13, C14, C15, C16, C17, C18, C19, C2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
