File: kikad/platy/platy.kicad_sch (KiCad schematic)
At the start: 31 parts, among them U1 ESP32-S3, U2 APS6404L-3SQRx-SN, U3 W25Q128JVS, U4 CC1101, Y1 40Mhz(+-10 ppm), Y2 Crystal

Commit message: Updated the schiematic
Parts:
- added C15, C18, C19, C21, C28: 0.1uF, symbol Device:C
- added C16, C17: 22uF, symbol Device:C
- added C20: 4.7uF, symbol Device:C
- added C22, C23: 220pF, symbol Device:C
- added C24, C25: 22pF, symbol Device:C
- added C26, C27: 200pF, symbol Device:C
- added C29: 1nF, symbol Device:C_Small
- added D2: LED, symbol Device:LED
- added J1: Conn_01x10, symbol Connector_Generic:Conn_01x10
- added J2: Conn_01x08, symbol Connector_Generic:Conn_01x08
- added JP1, JP2: Jumper_2_Bridged, symbol Jumper:Jumper_2_Bridged
- added L3, L4: 560nH, symbol Device:L
- added R10: 10K, symbol Device:R
- added R11: 1.6K, symbol Device:R
- added R12, R20: 1K, symbol Device:R_Small
- added R13, R14, R15, R16, R17: 100, symbol Device:R_Small
- added R18, R19: 10K, symbol Device:R_Small
- added R21, R22: 4.7K, symbol Device:R_Small
- added R9: 20K, symbol Device:R
- added SW1: SW_DPST, symbol Switch:SW_DPST
- added U5: PN5321A3HN_C1xx, Package_DFN_QFN:HVQFN-40-1EP_6x6mm_P0.5mm_EP4.1x4.1mm, symbol RF_NFC:PN5321A3HN_C1xx
- added Y3: 27.12Mhz, symbol Device:Crystal
Connections:
- net GND: now also C15.2, C16.2, C17.1, C18.2, C19.1, C20.2, C21.2, C22.2, C23.1, C24.2, C25.2, C26.1, C26.2, C27.1, C27.2, C28.2, D2.1 (K), R18.1, R19.2, R9.2, U5.1 (DVSS), U5.11 (AVSS), U5.18 (TESTEN), U5.3 (TVSS1), U5.41 (AVSS), U5.7 (TVSS2)
- new net: J2.2 (Pin_2), R14.2
- new net: C16.1, U5.14 (OSCIN), Y3.2
- new net: L4.1, U5.6 (TX2)
- new net: C23.2, C25.1, L4.2, R11.2
- new net: J2.1 (Pin_1), R13.2
- new net: J2.3 (Pin_3), R15.2
- new net: J2.4 (Pin_4), R16.2
- new net: J2.7 (Pin_7), R17.2
- new net: C29.1, R12.1, U5.10 (RX)
- new net: C17.2, U5.15 (OSCOUT), Y3.1
- new net: C15.1, U5.23 (PVDD)
- new net: L3.1, U5.4 (TX1)
- new net: C18.1, U5.40 (VBAT)
- new net: C20.1, C21.1, U5.5 (TVDD)
- new net: C19.2, U5.8 (AVDD)
- new net: C28.1, R12.2, U5.9 (VMID)
- new net: C22.1, C24.1, L3.2
- new net: C29.2, R11.1
- new net: D2.2 (A), R20.2
- new net: JP1.2 (B), JP2.2 (B)
- new net: SW1.1, SW1.3
- new net AUX1: J1.10 (Pin_10), U5.12 (AUX1)
- new net AUX2: J1.9 (Pin_9), U5.13 (AUX2)
- new net DBG_RX: J1.8 (Pin_8), U5.24 (P30/UART_RX)
- new net DBG_TX: J1.7 (Pin_7), U5.31 (P31/UART_TX)
- new net I0: JP1.1 (A), R18.2, SW1.2, U5.16 (I0)
- new net I1: JP2.1 (A), R19.1, SW1.4, U5.17 (I1)
- new net INT0: J1.6 (Pin_6), U5.32 (P32_INT0)
- new net INT1: J1.5 (Pin_5), U5.33 (P33_INT1)
- new net IRQ: R17.1
- new net MISO: R14.1, U5.29 (MISO/P71)
- new net MOSI/SDA/TX: R15.1, U5.28 (MOSI/SDA/HSU_TX)
- new net RSTOUT_N: J2.8 (Pin_8)
- new net RSTPD_N: J1.1 (Pin_1), R10.2, R9.1, U5.38 (~{RSTPD})
- new net SCK: R13.1, U5.30 (SCK/P72)
- new net SIGCLK: J1.4 (Pin_4), U5.34 (SIC_CLK/P34)
- new net SIGIN: J1.2 (Pin_2), U5.36 (SIGIN)
- new net SIGOUT: J1.3 (Pin_3), U5.35 (SIGOUT)
- new net SSEL/SCL/RX: R16.1, U5.27 (NSS/P50_SCL/HSU_RX)
Other:
- note added: "PN532"
- note added: "power 3v3"
- note added: "power supply 5v"

Commit message: wroom
Parts:
- added C? (x2): 10uF, symbol Device:C
- added C?: 100nF, symbol Device:C
- added D?: SS14, Diode_SMD:D_SMA, symbol Diode:SS14
- added D?: LED, symbol Device:LED
- added D?: SP0503BAHT, Package_TO_SOT_SMD:SOT-143, symbol Power_Protection:SP0503BAHT
- added J?: USB_C_Receptacle_USB2.0_16P, symbol Connector:USB_C_Receptacle_USB2.0_16P
- added R? (x2): R, symbol Device:R
- added R?: 220 ohm, symbol Device:R
- added U?: ESP32-S3-WROOM-1, RF_Module:ESP32-S3-WROOM-1, symbol RF_Module:ESP32-S3-WROOM-1
- added U?: AMS1117-3.3, Package_TO_SOT_SMD:SOT-223-3_TabPin2, symbol Regulator_Linear:AMS1117-3.3
Connections:
- net GND: now also C?.2, C?.2, C?.2, D?.1 (A), D?.1 (K), J?.A1 (GND), J?.A12 (GND), J?.B1 (GND), J?.B12 (GND), J?.SH (SHIELD), U?.1 (GND), U?.1 (GND), U?.40 (GND), U?.41 (GND)
- new net: D?.2 (A), D?.4 (K), J?.A4 (VBUS), J?.A9 (VBUS), J?.B4 (VBUS), J?.B9 (VBUS)
- new net: D?.2 (A), R?.2
- new net: J?.A5 (CC1), R?.1
- new net: J?.B5 (CC2), R?.1
- new net 3.3V: C?.1, C?.1, U?.2 (3V3), U?.2 (VO)
- new net 5V: C?.1, R?.1, U?.3 (VI)
- new net USB_D+: D?.2 (K), J?.A6 (D+), J?.B6 (D+), U?.14 (USB_D+)
- new net USB_D-: D?.3 (K), J?.A7 (D-), J?.B7 (D-), U?.13 (USB_D-)
- no-connect marks 0 -> 2
Other:
- note added: "U0RXD"
- note added: "U0TXD"

Commit message: added the mosfet and made the changes in the component
Parts:
- removed C? (x2): 10uF, symbol Device:C
- removed C?: 100nF, symbol Device:C
- removed D?: SS14, Diode_SMD:D_SMA, symbol Diode:SS14
- removed D?: LED, symbol Device:LED
- removed D?: SP0503BAHT, Package_TO_SOT_SMD:SOT-143, symbol Power_Protection:SP0503BAHT
- removed J?: USB_C_Receptacle_USB2.0_16P, symbol Connector:USB_C_Receptacle_USB2.0_16P
- removed R? (x2): R, symbol Device:R
- removed R?: 220 ohm, symbol Device:R
- removed U?: ESP32-S3-WROOM-1, RF_Module:ESP32-S3-WROOM-1, symbol RF_Module:ESP32-S3-WROOM-1
- removed U?: AMS1117-3.3, Package_TO_SOT_SMD:SOT-223-3_TabPin2, symbol Regulator_Linear:AMS1117-3.3
- added C30, C32: 10uF, symbol Device:C
- added C31: 100nF, symbol Device:C
- added D3: LED, symbol Device:LED
- added D4: SP0503BAHT, Package_TO_SOT_SMD:SOT-143, symbol Power_Protection:SP0503BAHT
- added D5: SS14, Diode_SMD:D_SMA, symbol Diode:SS14
- added J3: USB_C_Receptacle_USB2.0_16P, symbol Connector:USB_C_Receptacle_USB2.0_16P
- added Q1, Q2: 2N7002, 2N7002:SOT95P240X111-3N, symbol 2N7002:2N7002
- added R23: 220 ohm, symbol Device:R
- added R24, R25: 5.1K, symbol Device:R
- added U6: AMS1117-3.3, Package_TO_SOT_SMD:SOT-223-3_TabPin2, symbol Regulator_Linear:AMS1117-3.3
- added U7: ESP32-S3-WROOM-1, RF_Module:ESP32-S3-WROOM-1, symbol RF_Module:ESP32-S3-WROOM-1
Connections:
- net miso is gone; now on net MISO: U1.18 (GPIO13), U4.2 (SO/GDO1)
- net mosi is gone; now on net MOSI/SDA/TX: U1.16 (GPIO11), U4.20 (SI)
- net sclk is gone; now on net SCK: U1.17 (GPIO12), U4.1 (SCLK)
- net CSn: now also U7.18 (IO10)
- net GND: now also C30.2, C31.2, C32.2, D3.1 (K), D4.1 (A), J3.A1 (GND), J3.A12 (GND), J3.B1 (GND), J3.B12 (GND), J3.SH (SHIELD), R24.2, R25.2, U6.1 (GND), U7.1 (GND), U7.40 (GND), U7.41 (GND)
- net MISO: now also U7.21 (IO13)
- net MOSI/SDA/TX: now also U7.19 (IO11)
- net SCK: now also U7.20 (IO12)
- net SSEL/SCL/RX: now also Q1.3, Q2.3, U7.17 (IO9)
- net USB_D+: now also D4.2 (K), J3.A6 (D+), J3.B6 (D+), U7.14 (USB_D+)
- net USB_D-: now also D4.3 (K), J3.A7 (D-), J3.B7 (D-), U7.13 (USB_D-)
- net VDD33: no longer U4.11 (AVDD2), U4.14 (AVDD3), U4.15 (AVDD4), U4.18 (DGUARD), U4.4 (DVDD), U4.9 (AVDD1)
- net +3V3: now reaches C15.1, U5.23 (PVDD)
- net +3V3: now also C19.2, C20.1, C21.1, JP1.2 (B), JP2.2 (B), R20.1, R21.1, R22.1, SW1.1, SW1.3, U4.11 (AVDD2), U4.14 (AVDD3), U4.15 (AVDD4), U4.18 (DGUARD), U4.4 (DVDD), U4.9 (AVDD1), U5.5 (TVDD), U5.8 (AVDD), C31.1, C32.1, Q1.1, Q2.1, U6.2 (VO), U7.2 (3V3)
- net +5V: now reaches C18.1, U5.40 (VBAT)
- net +5V: now also R10.1, C30.1, D5.1 (K), R23.1, U6.3 (VI)
- net at R21.2: now also Q2.2
- net at R22.2: now also Q1.2
- new net: D4.4 (K), D5.2 (A), J3.A4 (VBUS), J3.A9 (VBUS), J3.B4 (VBUS), J3.B9 (VBUS)
- new net: D3.2 (A), R23.2
- new net: J3.A5 (CC1), R24.1
- new net: J3.B5 (CC2), R25.1
Other:
- note added: "ESP32 S3 WROOM 1"
- note added: "USB TYPE C"
- note added: "VOLTAGE REGULATOR"

Commit message: ir
Parts:
- added C? (x2): 0.1uF, symbol Device:C
- added C?: 470pF, symbol Device:C
- added C?: 10pF, symbol Device:C
- added C?: 100nF, symbol Device:C
- added D?: BPW34, OptoDevice:Osram_DIL2_4.3x4.65mm_P5.08mm, symbol Sensor_Optical:BPW34
- added D?: LED, symbol Device:LED
- added Q?: Q_NPN, symbol Device:Q_NPN
- added R? (x4): 10k, symbol Device:R
- added R?: 220 ohm, symbol Device:R
- added R? (x2): 100 ohm, symbol Device:R
- added R? (x2): 100k, symbol Device:R
- added SW?: SW_Push(Boot), symbol Switch:SW_Push
- added SW?: SW_Push(EN), symbol Switch:SW_Push
- added U? (x3): TLV9062, symbol Amplifier_Operational:TLV9062
- added U? (x2): LM393, symbol Comparator:LM393
Connections:
- net +3V3: now also D?.1 (K), R?.1, R?.1, R?.1, R?.1, R?.2, U?.8 (V+), U?.8 (V+)
- net GND: now also C?.2, C?.2, C?.2, Q?.E, R?.2, U?.2 (-), U?.3 (+), U?.4 (V-), U?.4 (V-), U?.5 (+)
- net BOOT: now reaches U7.27 (IO0)
- net BOOT: now also C?.1, R?.2, SW?.1, SW?.2
- net EN: now reaches U7.3 (EN)
- net EN: now also C?.1, C?.1, R?.2, R?.2, SW?.1, SW?.2
- net OUT: now reaches U7.32 (IO39)
- net OUT: now also R?.2, U?.1
- net IN: now reaches U7.5 (IO5)
- net IN: now also R?.1
- new net: C?.1, D?.2 (A), R?.1, U?.2 (-)
- new net: C?.1, C?.2, R?.2, U?.1
- new net: Q?.B, R?.1, R?.2
- new net: C?.2, R?.1, U?.6 (-)
- new net: R?.2, U?.3 (+), U?.7
- new net: D?.1 (K), Q?.C
- new net: D?.2 (A), R?.1
Other:
- note added: "BOOT AND ENABLE"

Commit message: updated schiematic and the added macro sd card
Parts:
- removed C? (x2): 0.1uF, symbol Device:C
- removed C?: 470pF, symbol Device:C
- removed C?: 10pF, symbol Device:C
- removed D?: BPW34, OptoDevice:Osram_DIL2_4.3x4.65mm_P5.08mm, symbol Sensor_Optical:BPW34
- removed D?: LED, symbol Device:LED
- removed Q?: Q_NPN, symbol Device:Q_NPN
- removed R? (x3): 10k, symbol Device:R
- removed R?: 220 ohm, symbol Device:R
- removed R? (x2): 100 ohm, symbol Device:R
- removed R? (x2): 100k, symbol Device:R
- removed SW?: SW_Push(Boot), symbol Switch:SW_Push
- removed SW?: SW_Push(EN), symbol Switch:SW_Push
- removed U? (x3): TLV9062, symbol Amplifier_Operational:TLV9062
- removed U? (x2): LM393, symbol Comparator:LM393
- added C33: 10pF, symbol Device:C
- added C34: 470pF, symbol Device:C
- added C35, C36: 0.1uF, symbol Device:C
- added C37, C44: 100nF, symbol Device:C_Small
- added C38, C41, C42: 100nF, symbol Device:C
- added C39, C40, C43: 220nF, symbol Device:C
- added D10, D11: 1N5822, Diode_THT:D_DO-201AD_P15.24mm_Horizontal, symbol Diode:1N5822
- added D6: BPW34, OptoDevice:Osram_DIL2_4.3x4.65mm_P5.08mm, symbol Sensor_Optical:BPW34
- added D7: LED, symbol Device:LED
- added D8: IR led, symbol Device:LED
- added D9: D_TVS, symbol Device:D_TVS
- added F1: Fuse, symbol Device:Fuse
- added J4: Conn_01x02_Socket, symbol Connector:Conn_01x02_Socket
- added J5: Micro_SD_Card, symbol Connector:Micro_SD_Card
- added L5, L6: 33uH, symbol Device:L
- added Q3: Q_NPN, symbol Device:Q_NPN
- added Q4: BC847, Package_TO_SOT_SMD:SOT-23, symbol Transistor_BJT:BC847
- added Q5: Q_PMOS_GSD, symbol Transistor_FET:Q_PMOS_GSD
- added R26: 220 ohm, symbol Device:R
- added R27, R29: 100 ohm, symbol Device:R
- added R28, R30, R37: 100k, symbol Device:R
- added R31, R32, R33: 10k, symbol Device:R
- added R34: R_Small, symbol Device:R_Small
- added R35: 100, symbol Device:R
- added R36, R40: 1K, symbol Device:R
- added R38: 1.68k, symbol Device:R
- added R39: 1k, symbol Device:R
- added SW2: SW_Push(Boot), symbol Switch:SW_Push
- added SW3: SW_Push(EN), symbol Switch:SW_Push
- added U10: TSOP382xx, OptoDevice:Vishay_MINICAST-3Pin, symbol Interface_Optical:TSOP382xx
- added U11: LM2596S-5, Package_TO_SOT_SMD:TO-263-5_TabPin3, symbol Regulator_Switching:LM2596S-5
- added U12: LM2596S-3.3, Package_TO_SOT_SMD:TO-263-5_TabPin3, symbol Regulator_Switching:LM2596S-3.3
- added U8: TLV9062, symbol Amplifier_Operational:TLV9062
- added U9: LM393, symbol Comparator:LM393
Connections:
- net +3V3: now also C42.1, C43.1, C44.1, D6.1 (K), J5.4 (VDD), L6.2, R29.2, R31.1, R32.1, R33.1, R34.2, R35.1, R38.2, R40.1, U8.8 (V+), U9.8 (V+)
- net +5V: now also C40.1, C41.1, L5.2, U11.4 (FB)
- net BOOT: now also C35.1, R32.2, SW2.1, SW2.2
- net EN: now also C36.1, R33.2, SW3.1, SW3.2
- net GND: now also C35.2, C36.2, C37.2, C38.2, C39.2, C40.2, C41.2, C42.2, C43.2, C44.2, D10.2 (A), D11.2 (A), D9.2 (A2), J5.6 (VSS), J5.SH (SHIELD), Q3.E, Q4.2 (E), R27.2, R37.2, R39.2, U10.2 (GND), U11.3 (GND), U11.5 (~{ON}/OFF), U12.3 (GND), U12.5 (~{ON}/OFF), U8.3 (+), U8.4 (V-), U8.5 (+), U9.2 (-), U9.4 (V-)
- net IN: now also R26.1
- net MISO: now also J5.7 (DAT0)
- net MOSI/SDA/TX: now also J5.3 (CMD)
- net OUT: now also R31.2, U9.1
- net SCK: now also J5.5 (CLK)
- net GPIO 4: now reaches U7.4 (IO4)
- net GPIO 4: now also C37.1, U10.1 (OUT)
- net gpio 6: now reaches U7.6 (IO6)
- net gpio 6: now also R36.2
- net CSN: now reaches U7.8 (IO15)
- net CSN: now also J5.2 (DAT3/CD), R40.2
- new net: D8.1 (K), Q4.3 (C)
- new net: D8.2 (A), R35.2
- new net: C33.2, C34.1, R28.2, U8.1
- new net: C34.2, R30.1, U8.6 (-)
- new net: R30.2, U8.7, U9.3 (+)
- new net: D7.1 (K), Q3.C
- new net: D7.2 (A), R29.1
- new net: Q3.B, R26.2, R27.1
- new net: R34.1, U10.3 (Vs)
- new net: Q4.1 (B), R36.1
- new net: D10.1 (K), L5.1, U11.2 (OUT)
- new net: D11.1 (K), L6.1, U12.2 (OUT)
- new net: R38.1, R39.1, U12.4 (FB)
- new net: C33.1, D6.2 (A), R28.1, U8.2 (-)
- new net: F1.2, Q5.3 (D)
- new net: Q5.1 (G), R37.1
- new net BAT+: F1.1, J4.1 (Pin_1)
- new net Gnd: J4.2 (Pin_2)
- new net Vin: C38.1, C39.1, D9.1 (A1), Q5.2 (S), U11.1 (VIN), U12.1 (VIN)
- no-connect marks 2 -> 4
Other:
- note added: "Battery"
- note added: "IR Transmitter"
- note added: "IR receiver"
- note added: "Macro SD card"
- moved on the sheet: C1, C10, C11, C12, C13, C14, C15, C16, C17, C18, C19, C2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

Commit message: joystick added and sorted out majority of erc errors
Parts:
- removed D3: LED, symbol Device:LED
- removed R23: 220 ohm, symbol Device:R
- added C32, C45, C48: 100nF, symbol Device:C
- added J6: Conn_01x05_Pin, symbol Connector:Conn_01x05_Pin
- gave numbers to parts that had none: 2
- renumbered C16 to C12, C17 to C13, C18 to C15, C19 to C16, C12 to C17, C13 to C18, C15 to C19, C28 to C20, C20 to C21, C29 to C22, C44 to C23, C21 to C24, C22 to C25, C23 to C26, C24 to C27, C25 to C28, C26 to C29, C27 to C30, C37 to C31, C30 to C36, C31 to C37, C32 to C44, C35 to C46, C36 to C47, D8 to D4, D4 to D5, D5 to D8, J5 to J1, J1 to J2, J2 to J3, J3 to J5, Q2 to Q1, Q1 to Q2, R9 to R11, R18 to R12, R19 to R13, R8 to R14, R12 to R15, R40 to R16, R20 to R17, R11 to R18, R15 to R19, R17 to R20, R35 to R21, R13 to R22, R16 to R24, R14 to R25, R34 to R32, R36 to R33, R24 to R34, R25 to R35, R32 to R40, R33 to R41, R21 to R8, R22 to R9, U7 to U10, U10 to U6, U6 to U7, Y3 to Y2, Y2 to Y3
Connections:
- net Gnd is gone; now on net GND: J4.2 (Pin_2)
- net +3V3: no longer C16.2, C19.1, C21.1, C23.1, C24.1, C37.1, C42.1, C43.1, C44.1, J1.4 (VDD), JP1.2 (B), JP2.2 (B), L6.2, Q1.1, Q2.1, R16.1, R17.1, R21.1, R32.2, R38.2, R40.1, R41.1, R8.1, R9.1, SW1.1, SW1.3, U10.2 (3V3), U4.11 (AVDD2), U4.14 (AVDD3), U4.15 (AVDD4), U4.18 (DGUARD), U4.4 (DVDD), U4.9 (AVDD1), U5.23 (PVDD), U5.5 (TVDD), U5.8 (AVDD), U7.2 (VO)
- net +5V: no longer C15.1, C36.1, U5.40 (VBAT), U7.3 (VI)
- net GND: now also C45.2, C48.2, J6.2 (Pin_2)
- net MISO: no longer U1.18 (GPIO13), U4.2 (SO/GDO1)
- net VDD33: no longer C10.1, C8.1, C9.1, L1.1
- net Vin: now also C32.1
- net at U1.2 (VDD3P3), U1.3 (VDD3P3): no longer C7.1, L1.2
- net GPIO 47: now reaches U10.24 (IO47)
- net GPIO 47: now also J6.4 (Pin_4)
- net GPIO 48: now reaches U10.25 (IO48)
- net GPIO 48: now also J6.5 (Pin_5)
- net GPIO 38: now reaches U10.31 (IO38)
- net GPIO 38: now also J6.3 (Pin_3)
- new net: C32.2, C36.1, U7.3 (VI)
- new net: C7.1, L1.2
- new net 3v3: C10.1, C15.1, C16.2, C19.1, C21.1, C23.1, C24.1, C37.1, C42.1, C43.1, C44.1, C45.1, C48.1, C8.1, C9.1, J1.4 (VDD), J6.1 (Pin_1), JP1.2 (B), JP2.2 (B), L1.1, L6.2, Q1.1, Q2.1, R16.1, R17.1, R21.1, R32.2, R38.2, R40.1, R41.1, R8.1, R9.1, SW1.1, SW1.3, U10.2 (3V3), U4.11 (AVDD2), U4.14 (AVDD3), U4.15 (AVDD4), U4.18 (DGUARD), U4.4 (DVDD), U4.9 (AVDD1), U5.23 (PVDD), U5.40 (VBAT), U5.5 (TVDD), U5.8 (AVDD), U7.2 (VO)
- new net miso: U1.18 (GPIO13), U4.2 (SO/GDO1)
- no-connect marks 4 -> 93
Other:
- note added: "JOYSTICK"
- moved on the sheet: C38, C39, C40, C41, C42, C43, D10, D11, D9, F1, J4, L5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
