File: kikad/platy/platy.kicad_sch (KiCad schematic)
At the start: 136 parts, among them J1 Micro_SD_Card, J2 Conn_01x10, J3 Conn_01x08, J4 Conn_01x02_Socket, J5 USB_C_Receptacle_USB2.0_16P, J6 Conn_01x05_Pin, Q1 2N7002, Q2 2N7002, Q3 Q_NPN, Q4 BC847, Q5 Q_PMOS_GSD, SW1 SW_DPST, SW2 SW_Push(Boot), SW3 SW_Push(EN), U1 ESP32-S3, U10 ESP32-S3-WROOM-1, U11 LM2596S-5, U12 LM2596S-3.3, U2 APS6404L-3SQRx-SN, U3 W25Q128JVS, U4 CC1101, U5 PN5321A3HN_C1xx, U6 TSOP382xx, U7 AMS1117-3.3, U8 TLV9062, U9 LM393, Y1 40Mhz(+-10 ppm), Y2 27.12Mhz, Y3 Crystal

Commit message: solved all erc errors and added connectors
Parts:
- added J7: Conn_01x09_Pin, symbol Connector:Conn_01x09_Pin
Connections:
- net 3v3: now also J7.1 (Pin_1), J7.3 (Pin_3)
- net GND: now also J7.2 (Pin_2)
- net MOSI/SDA/TX: now also J7.9 (Pin_9)
- net SCK: now also J7.5 (Pin_5)
- net LCD_DC: now reaches U10.10 (IO17)
- net LCD_DC: now also J7.4 (Pin_4)
- net LCD_RST: now reaches U10.12 (IO8)
- net LCD_RST: now also J7.8 (Pin_8)
- net LCD_CS: now reaches U10.22 (IO14)
- net LCD_CS: now also J7.6 (Pin_6)
- no-connect marks 93 -> 92
Other:
- note added: "EN"
- note added: "GND"
- note added: "VCC"

Commit message: made changes told  by the mentors
Parts:
- added AE1: 50ohm, symbol Device:Antenna
- added C49, C54: 3.9pF, symbol Device:C
- added C50: 8.2pF, symbol Device:C
- added C51: 5.6pF, symbol Device:C
- added C52, C53: 220pF, symbol Device:C
- added C55, C56: 100nF, symbol Device:C
- added L7, L9, L?: 27nH, symbol Device:L
- added L8: 22nH, symbol Device:L
- added U13: CR2013-MI2120, Display:CR2013-MI2120, symbol Driver_Display:CR2013-MI2120
- C14: value C -> 100nF
- C17, C18: value C -> 27pF
- R32: value R_Small -> 300ohms
- Y3: value Crystal -> 26MHz
Connections:
- net +3V3: no longer R36.1
- net 3v3: now also R36.1, C55.1, C56.1, U13.1 (VCC)
- net BOOT: no longer C46.1, SW2.1
- net EN: no longer C47.1, SW3.1
- net GND: now also C49.1, C50.2, C51.2, C53.2, C55.2, C56.2, U13.2 (GND)
- net GPIO 38: no longer J6.3 (Pin_3)
- net GPIO 47: no longer J6.4 (Pin_4)
- net GPIO 48: no longer J6.5 (Pin_5)
- net MOSI/SDA/TX: no longer J1.3 (CMD), J7.9 (Pin_9), U1.16 (GPIO11), U10.19 (IO11), U4.20 (SI), U5.28 (MOSI/SDA/HSU_TX)
- net SSEL/SCL/RX: no longer U10.17 (IO9), U5.27 (NSS/P50_SCL/HSU_RX)
- net at U4.12 (RF_P): now also C54.2, L?.2
- net at U4.13 (RF_N): now also C49.2, L7.1
- new net: C54.1, L7.2, L8.1
- new net: C50.1, L8.2, L9.1
- new net: C51.1, C52.2, L9.2
- new net: C47.1, SW3.1
- new net: C46.1, SW2.1
- new net: AE1.1 (A), C52.1
- new net: C53.1, L?.1
- new net MOSI: J1.3 (CMD), J7.9 (Pin_9), U1.16 (GPIO11), U10.19 (IO11), U4.20 (SI), U5.28 (MOSI/SDA/HSU_TX)
- new net SSEL: U10.17 (IO9), U5.27 (NSS/P50_SCL/HSU_RX)
- no-connect marks 92 -> 88
Other:
- moved on the sheet: C35, C45, R36, U10

Commit message: added the nrf module and made the change in the schiematic
Parts:
- added C57: 33nF, symbol Device:C
- added C58, C59: 22uF, symbol Device:C_Small
- added C60: 1.5uF, symbol Device:C_Small
- added C61: 4.7pF, symbol Device:C_Small
- added C62: 1pF, symbol Device:C_Small
- added C63: 22nF, symbol Device:C_Small
- added C64: 1nF, symbol Device:C_Small
- added C65: 10nF, symbol Device:C_Small
- added L10: 3.9nH, symbol Device:L
- added L11: 8.2nH, symbol Device:L
- added L12: 2.7nH, symbol Device:L
- added R23: 22K, symbol Device:R_Small
- added R42: 1M, symbol Device:R_Small
- added U14: NRF24L01, Package_DFN_QFN:QFN-20-1EP_4x4mm_P0.5mm_EP2.5x2.5mm, symbol RF:NRF24L01
- added Y4: 16Mhz, symbol Device:Crystal
- gave numbers to parts that had none: 1
Connections:
- net 3v3: now also C64.1, C65.1, U14.15 (VDD), U14.18 (VDD), U14.7 (VDD)
- net GND: now also C57.2, C58.2, C59.1, C61.2, C62.1, C63.2, C64.2, C65.2, R23.2, U14.14 (VSS), U14.17 (VSS), U14.20 (VSS), U14.8 (VSS)
- net IRQ: now also U10.28 (IO35), U14.6 (IRQ)
- net MISO: now also U14.5 (MISO)
- net MOSI: now also U14.4 (MOSI)
- net SCK: now also U14.3 (SCK)
- net CE: now reaches U10.23 (IO21)
- net CE: now also U14.1 (CE)
- net csn_nrf: now reaches U10.9 (IO16)
- net csn_nrf: now also U14.2 (CSN)
- new net: C58.1, R42.1, U14.10 (XC1), Y4.1
- new net: C59.2, R42.2, U14.9 (XC2), Y4.2
- new net: C60.1, L10.2
- new net: C60.2, C62.2
- new net: C57.1, U14.19 (DVDD)
- new net: R23.1, U14.16 (IREF)
- new net: L11.1, L12.1, U14.12 (ANT1)
- new net: C61.1, C63.1, L12.2, U14.11 (VDD_PA)
- new net: L10.1, L11.2, U14.13 (ANT2)
- no-connect marks 88 -> 85
Other:
- note added: "50ohm, RF I/O"
- note added: "NRf24L01"
- moved on the sheet: JP1, JP2

Commit message: made the changes and the added for the display
Parts:
- removed C33: 10pF, symbol Device:C
- removed C34: 470pF, symbol Device:C
- removed D6: BPW34, OptoDevice:Osram_DIL2_4.3x4.65mm_P5.08mm, symbol Sensor_Optical:BPW34
- removed J6: Conn_01x05_Pin, symbol Connector:Conn_01x05_Pin
- removed R28, R30: 100k, symbol Device:R
- removed R31: 10k, symbol Device:R
- removed U13: CR2013-MI2120, Display:CR2013-MI2120, symbol Driver_Display:CR2013-MI2120
- removed U8: TLV9062, symbol Amplifier_Operational:TLV9062
- removed U9: LM393, symbol Comparator:LM393
- added C66: 1uF, symbol Device:C_Small
- added J6: Conn_01x04_Pin, symbol Connector:Conn_01x04_Pin
- added J8: Conn_01x14_Socket, symbol Connector:Conn_01x14_Socket
- F1: value Fuse -> 2A
Connections:
- net +3V3 is gone; now on net 3v3: R29.2
- net miso is gone; now on net MISO: U1.18 (GPIO13), U4.2 (SO/GDO1)
- net +5V: no longer R10.1
- net 3v3: now also R10.1, C66.1, J6.1 (Pin_1), J8.1 (Pin_1), J8.9 (Pin_9)
- net BOOT: now also C46.1, SW2.1; no longer R40.2, SW2.2
- net CSN: now also J8.11 (Pin_11)
- net EN: now also C47.1, SW3.1; no longer R41.2, SW3.2
- net GND: now also C66.2, J6.2 (Pin_2), J8.2 (Pin_2)
- net MISO: now also J8.12 (Pin_12), J8.8 (Pin_8)
- net MOSI: now also J8.13 (Pin_13), J8.6 (Pin_6)
- net SCK: now also J8.10 (Pin_10), J8.7 (Pin_7)
- net cs_tht: now reaches U10.15 (IO3)
- net cs_tht: now also J8.3 (Pin_3)
- net Vrx: now reaches U10.29 (IO36)
- net Vrx: now also J6.3 (Pin_3)
- net Vry: now reaches U10.30 (IO37)
- net Vry: now also J6.4 (Pin_4)
- net irq_tht: now reaches U10.34 (IO41)
- net irq_tht: now also J8.14 (Pin_14)
- net d/c: now reaches U10.38 (IO2)
- net d/c: now also J8.5 (Pin_5)
- net reset: now reaches U10.7 (IO7)
- net reset: now also J8.4 (Pin_4)
- new net: R41.2, SW3.2
- new net: R40.2, SW2.2
- no-connect marks 85 -> 79
Other:
- note added: "ANTENA"
- note added: "DISPLAY THT"
- moved on the sheet: C48, D2, F1, J2, J3, J7, Q1, Q2, Q5, R12, R13, R17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

Commit message: resolved errors in schematic
Parts:
- added J9: Conn_02x04_Odd_Even, symbol Connector_Generic:Conn_02x04_Odd_Even
Connections:
- net 3v3: now also J9.2 (Pin_2)
- net CE: now also U10.35 (IO42), J9.3 (Pin_3)
- net GND: now also C32.1, C35.1, R36.2, SW2.1, SW3.1, U10.27 (IO0), U10.3 (EN), J9.1 (Pin_1)
- net IRQ: now also U10.26 (IO45), J9.8 (Pin_8)
- net MISO: now also J9.7 (Pin_7); no longer U1.18 (GPIO13)
- net MOSI: now also J9.6 (Pin_6); no longer J1.3 (CMD), J7.9 (Pin_9), U1.16 (GPIO11), U14.4 (MOSI)
- net SCK: now also J9.5 (Pin_5); no longer J1.5 (CLK), U1.17 (GPIO12), U14.3 (SCK)
- net Vin: now also C32.2, C36.1, U7.3 (VI); no longer C32.1
- net csn_nrf: no longer U10.9 (IO16)
- net at R41.2, SW3.2: now also C47.1
- net at R40.2, SW2.2: now also C46.1
- removed net BOOT: C46.1, SW2.1, U10.27 (IO0)
- removed net EN: C35.1, C47.1, R36.2, SW3.1, U10.3 (EN)
- new net CNS: J9.4 (Pin_4), U10.9 (IO16)
- new net Mosi: J1.3 (CMD), U14.4 (MOSI)
- new net clk: J1.5 (CLK), U14.3 (SCK)
- new net miso: U1.18 (GPIO13)
- new net mosi: J7.9 (Pin_9), U1.16 (GPIO11)
- new net sclk: U1.17 (GPIO12)
- no-connect marks 79 -> 77
Other:
- note added: "DISPLAY TFT"
- note added: "TSOP38238"
- note removed: "DISPLAY THT"
- note removed: "IR receiver"
- note removed: "SCLK"
- moved on the sheet: AE1, C12, C13, C14, C15, C16, C17, C18, C19, C20, C21, C22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
