File: kicad/platy/platy.kicad_sch (KiCad schematic)
At the start: 86 parts, among them J1 Conn_01x04_Socket, J2 Conn_01x02_Socket, J5 USB_C_Receptacle_USB2.0_16P, J6 Conn_01x04_Pin, J8 Conn_01x14_Socket, J9 Conn_02x04_Odd_Even, Q4 BC847, Q5 Q_PMOS_GSD, SW1 SW_DPST, SW2 SW_Push(Boot), SW3 SW_Push(EN), U10 ESP32-S3-WROOM-1, U4 CC1101, U5 PN5321A3HN_C1xx, U6 TSOP382xx, U7 AMS1117-3.3, Y2 27.12Mhz, Y3 26MHz

Commit message: Completed the most of the routing
Parts:
- SW1: footprint (none) -> Button_Switch_SMD:SW_DIP_SPSTx02_Slide_6.7x6.64mm_W6.73mm_P2.54mm_LowProfile_JPin
Connections:
- net 3v3: no longer J8.9 (Pin_9)
- net MISO: now also J8.9 (Pin_9); no longer J8.8 (Pin_8)
- net SSEL/SCL/RX: now also R8.2, R9.2
- net led: now reaches U10.39 (IO1)
- net led: now also J8.8 (Pin_8)
- no-connect marks 15 -> 14
Changed lines of the file:
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@@
 	)
 	(no_connect
-		(at 304.8 166.37)
-	)
-	(no_connect
 		(at 99.06 212.09)
 	)
@@
 	(wire
 		(pts
-			(xy 304.8 166.37) (xy 318.77 166.37)
-		)
-		(stroke
-			(width 0)
-			(type default)
-		)
-	)
-	(wire
-		(pts
 			(xy 114.3 55.88) (xy 119.38 55.88)
 		)
@@
 	(wire
 		(pts
+			(xy 203.2 295.91) (xy 213.36 295.91)
+		)
+		(stroke
+			(width 0)
+			(type default)
+		)
+	)
+	(wire
+		(pts
 			(xy 213.36 203.2) (xy 219.71 203.2)
 		)
@@
 	(wire
 		(pts
+			(xy 201.93 271.78) (xy 212.09 271.78)
+		)
+		(stroke
+			(width 0)
+			(type default)
+		)
+	)
+	(wire
+		(pts
 			(xy 212.09 58.42) (xy 212.09 60.96)
 		)
@@
 	(wire
 		(pts
+			(xy 303.53 166.37) (xy 318.77 166.37)
+		)
+		(stroke
+			(width 0)
+			(type default)
+		)
+	)
+	(wire
+		(pts
 			(xy 160.02 213.36) (xy 162.56 213.36)
 		)
@@
 		)
 	)
-	(label "MISO"
-		(at 297.18 55.88 180)
-		(effects
-			(font
-				(size 1.27 1.27)
-			)
-			(justify right bottom)
-		)
-	)
 	(label "SD_cs"
 		(at 331.47 39.37 180)
@@
 		)
 	)
+	(label "MISO"
+		(at 297.18 58.42 180)
+		(effects
+			(font
+				(size 1.27 1.27)
+			)
+			(justify right bottom)
+		)
+	)
 	(label "3v3"
 		(at 297.18 38.1 180)
@@
 		)
 	)
+	(label "led"
+		(at 297.18 55.88 180)
+		(effects
+			(font
+				(size 1.27 1.27)
+			)
+			(justify right bottom)
+		)
+	)
 	(label "BAT+"
 		(at 377.19 340.36 180)
@@
 		)
 	)
+	(label "led"
+		(at 303.53 166.37 180)
+		(effects
+			(font
+				(size 1.27 1.27)
+			)
+			(justify right bottom)
+		)
+	)
 	(label "USB_D+"
 		(at 322.58 330.2 0)
@@
 	)
 	(label "3v3"
-		(at 297.18 58.42 180)
-		(effects
-			(font
-				(size 1.27 1.27)
-			)
-			(justify right bottom)
-		)
-	)
-	(label "3v3"
 		(at 111.76 179.07 0)
 		(effects
@@
 			)
 		)
-		(property "Footprint" ""
+		(property "Footprint" "Button_Switch_SMD:SW_DIP_SPSTx02_Slide_6.7x6.64mm_W6.73mm_P2.54mm_LowProfile_JPin"
 			(at 74.93 306.07 0)
 			(hide yes)

Commit message: made the second ertation of the pcb
Changed lines of the file:
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@@
 	)
 	(junction
-		(at 201.93 260.35)
-		(diameter 0)
-		(color 0 0 0 0)
-	)
-	(junction
 		(at 339.09 134.62)
 		(diameter 0)
@@
 	)
 	(junction
-		(at 203.2 284.48)
-		(diameter 0)
-		(color 0 0 0 0)
-	)
-	(junction
 		(at 114.3 64.77)
 		(diameter 0)
@@
 	(wire
 		(pts
-			(xy 203.2 284.48) (xy 203.2 289.56)
-		)
-		(stroke
-			(width 0)
-			(type default)
-		)
-	)
-	(wire
-		(pts
 			(xy 135.89 87.63) (xy 142.24 87.63)
 		)
@@
 	(wire
 		(pts
-			(xy 205.74 289.56) (xy 205.74 290.83)
-		)
-		(stroke
-			(width 0)
-			(type default)
-		)
-	)
-	(wire
-		(pts
 			(xy 201.93 256.54) (xy 201.93 260.35)
 		)
@@
 	(wire
 		(pts
-			(xy 201.93 266.7) (xy 204.47 266.7)
-		)
-		(stroke
-			(width 0)
-			(type default)
-		)
-	)
-	(wire
-		(pts
 			(xy 62.23 36.83) (xy 62.23 40.64)
 		)
@@
 	(wire
 		(pts
-			(xy 201.93 260.35) (xy 201.93 266.7)
-		)
-		(stroke
-			(width 0)
-			(type default)
-		)
-	)
-	(wire
-		(pts
 			(xy 208.28 90.17) (xy 214.63 90.17)
 		)
@@
 		)
 		(stroke
-			(width 0)
-			(type default)
-		)
-	)
-	(wire
-		(pts
-			(xy 203.2 289.56) (xy 205.74 289.56)
-		)
-		(stroke

Commit message: updated pcb
Parts:
- added J3: Conn_Coaxial, Connector_Coaxial:U.FL_Molex_MCRF_73412-0110_Vertical, symbol Connector:Conn_Coaxial
- AE1: footprint RF_Antenna:Texas_SWRA416_868MHz_915MHz -> Connector_Coaxial:SMA_Amphenol_132134_Vertical
- J5: footprint Connector_USB:USB_C_Receptacle_HRO_TYPE-C-31-M-12 -> Connector_USB:USB_C_Receptacle_GCT_USB4105-xx-A_16P_TopMnt_Horizontal
- Y2, Y3: footprint Crystal:Crystal_HC49-U_Vertical -> Crystal:Crystal_SMD_5032-2Pin_5.0x3.2mm
Connections:
- net GND: now also J3.1 (In), J3.2 (Ext)
Changed lines of the file:
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@@
 	)
 	(junction
-		(at 213.36 209.55)
-		(diameter 0)
-		(color 0 0 0 0)
-	)
-	(junction
 		(at 72.39 36.83)
 		(diameter 0)
@@
 	)
 	(junction
+		(at 213.36 209.55)
+		(diameter 0)
+		(color 0 0 0 0)
+	)
+	(junction
 		(at 59.69 248.92)
 		(diameter 0)
@@
 	(wire
 		(pts
+			(xy 224.79 215.9) (xy 224.79 212.09)
+		)
+		(stroke
+			(width 0)
+			(type default)
+		)
+	)
+	(wire
+		(pts
 			(xy 146.05 214.63) (xy 146.05 215.9)
 		)
@@
 	(wire
 		(pts
+			(xy 224.79 212.09) (xy 238.76 212.09)
+		)
+		(stroke
+			(width 0)
+			(type default)
+		)
+	)
+	(wire
+		(pts
 			(xy 349.25 191.77) (xy 383.54 191.77)
 		)
@@
 	(wire
 		(pts
-			(xy 213.36 215.9) (xy 219.71 215.9)
+			(xy 213.36 215.9) (xy 224.79 215.9)
 		)
 		(stroke
@@
 	(wire
 		(pts
-			(xy 213.36 203.2) (xy 213.36 209.55)
-		)
-		(stroke
-			(width 0)
-			(type default)
-		)
-	)
-	(wire
-		(pts
 			(xy 297.18 45.72) (xy 307.34 45.72)
 		)
@@
 	(wire
 		(pts
-			(xy 213.36 209.55) (xy 213.36 215.9)
+			(xy 213.36 203.2) (xy 213.36 209.55)
 		)
 		(stroke
@@
 	(wire
 		(pts
-			(xy 74.93 44.45) (xy 74.93 36.83)
+			(xy 196.85 209.55) (xy 213.36 209.55)
 		)
 		(stroke
@@
 	(wire
 		(pts
-			(xy 139.7 212.09) (xy 147.32 212.09)
+			(xy 74.93 44.45) (xy 74.93 36.83)
 		)
 		(stroke
@@
 	(wire
 		(pts
-			(xy 349.25 161.29) (xy 397.51 161.29)
+			(xy 139.7 212.09) (xy 147.32 212.09)
 		)
 		(stroke
@@
 	(wire
 		(pts
-			(xy 299.72 184.15) (xy 318.77 184.15)
+			(xy 349.25 161.29) (xy 397.51 161.29)
 		)
 		(stroke
@@
 	(wire
 		(pts
-			(xy 213.36 209.55) (xy 219.71 209.55)
+			(xy 299.72 184.15) (xy 318.77 184.15)
 		)
 		(stroke
@@
 	(wire
 		(pts
+			(xy 233.68 203.2) (xy 233.68 205.74)
+		)
+		(stroke
+			(width 0)
+			(type default)
+		)
+	)
+	(wire
+		(pts
 			(xy 213.36 219.71) (xy 196.85 219.71)
 		)
@@
 	(wire
 		(pts
-			(xy 196.85 209.55) (xy 213.36 209.55)
-		)
-		(stroke
-			(width 0)
-			(type default)
-		)
-	)
-	(wire
-		(pts
 			(xy 298.45 204.47) (xy 318.77 204.47)
 		)
@@
 	(wire
 		(pts
-			(xy 213.36 203.2) (xy 219.71 203.2)
+			(xy 213.36 203.2) (xy 233.68 203.2)
 		)
 		(stroke
@@
 	(wire
 		(pts
+			(xy 213.36 209.55) (xy 213.36 215.9)
+		)
+		(stroke
+			(width 0)
+			(type default)
+		)
+	)
+	(wire
+		(pts
 			(xy 389.89 43.18) (xy 400.05 43.18)
 		)
@@
 	(wire
 		(pts
+			(xy 238.76 212.09) (xy 238.76 210.82)
+		)
+		(stroke
+			(width 0)
+			(type default)
+		)
+	)
+	(wire
+		(pts
 			(xy 72.39 36.83) (xy 74.93 36.83)
 		)
@@
 			)
 		)
-		(property "Footprint" "Crystal:Crystal_HC49-U_Vertical"
+		(property "Footprint" "Crystal:Crystal_SMD_5032-2Pin_5.0x3.2mm"
 			(at 114.3 59.69 0)
 			(hide yes)
@@
 	)
 	(symbol
+		(lib_id "Connector:Conn_Coaxial")
+		(at 238.76 205.74 0)
+		(unit 1)
+		(body_style 1)
+		(exclude_from_sim no)
+		(in_bom yes)
+		(on_board yes)
+		(in_pos_files yes)
+		(dnp no)
+		(fields_autoplaced yes)
+		(property "Reference" "J3"
+			(at 242.57 204.7631 0)
+			(show_name no)
+			(do_not_autoplace no)
+			(effects
+				(font
+					(size 1.27 1.27)
+				)
+				(justify left)
+			)
+		)
+		(property "Value" "Conn_Coaxial"
+			(at 242.57 207.3031 0)
+			(show_name no)
+			(do_not_autoplace no)
+			(effects
+				(font
+					(size 1.27 1.27)
+				)
+				(justify left)
+			)
+		)
+		(property "Footprint" "Connector_Coaxial:U.FL_Molex_MCRF_73412-0110_Vertical"
+			(at 238.76 205.74 0)
+			(hide yes)
+			(show_name no)
+			(do_not_autoplace no)
+			(effects
+				(font
+					(size 1.27 1.27)
+				)
+			)
+		)
+		(property "Datasheet" ""
+			(at 238.76 205.74 0)
+			(hide yes)
+			(show_name no)
+			(do_not_autoplace no)
+			(effects
+				(font
+					(size 1.27 1.27)
+				)
+			)
+		)
+		(property "Description" "coaxial connector (BNC, SMA, SMB, SMC, Cinch/RCA, LEMO, ...)"
+			(at 238.76 205.74 0)
+			(hide yes)
+			(show_name no)
+			(do_not_autoplace no)
+			(effects
+				(font
+					(size 1.27 1.27)
+				)
+			)
+		)
+		(pin "2"
+		)
+		(pin "1"
+		)
+		(instances
+			(project "platy"
+				(path "/d735ea85-ad76-451c-86ef-ab784456e68b"
+					(reference "J3")
+					(unit 1)
+				)
+			)
+		)
+	)
+	(symbol
 		(lib_id "power:PWR_FLAG")
 		(at 311.15 274.32 90)
@@
 			)
 		)
-		(property "Footprint" "RF_Antenna:Texas_SWRA416_868MHz_915MHz"
+		(property "Footprint" "Connector_Coaxial:SMA_Amphenol_132134_Vertical"
 			(at 142.24 129.54 0)
 			(hide yes)
@@
 			)
 		)
-		(property "Footprint" "Crystal:Crystal_HC49-U_Vertical"
+		(property "Footprint" "Crystal:Crystal_SMD_5032-2Pin_5.0x3.2mm"
 			(at 78.74 248.92 0)
 			(hide yes)
@@
 			)
 		)
-		(property "Footprint" "Connector_USB:USB_C_Receptacle_HRO_TYPE-C-31-M-12"
+		(property "Footprint" "Connector_USB:USB_C_Receptacle_GCT_USB4105-xx-A_16P_TopMnt_Horizontal"
 			(at 297.18 327.66 0)
 			(hide yes)

Commit message: changes the made in the routing and in the schiematic and also in the value in the component
Parts:
- C12, C13: value 22uF -> 22pF
Connections:
- net 5V is gone; now on net 3v3: D8.1 (K)
- net CE: no longer U10.35 (IO42)
- net IRQ: no longer U10.26 (IO45)
- net GDO0: now reaches U4.6 (GDO0)
- net GDO0: now also U10.26 (IO45)

Commit message: corrected the boot and the enable and other things also
Connections:
- net GND: no longer C35.1, R36.2, U10.27 (IO0), U10.3 (EN)
- net EN: now reaches C47.1, R41.2, SW3.2
- net EN: now also C35.1, R36.2, U10.3 (EN)
- net BOOT: now reaches C46.1, R40.2, SW2.2
- net BOOT: now also U10.27 (IO0)
- net gdo2: now reaches U4.3 (GDO2)
- net gdo2: now also U10.16 (IO46)
- no-connect marks 14 -> 12
Changed lines of the file:
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@@
 	)
 	(no_connect
-		(at 379.73 199.39)
-	)
-	(no_connect
 		(at 151.13 245.11)
 	)
@@
 		(at 308.61 342.9)
 	)
-	(no_connect
-		(at 38.1 67.31)
-	)
 	(wire
 		(pts
@@
 	(wire
 		(pts
-			(xy 38.1 67.31) (xy 52.07 67.31)
-		)
-		(stroke
-			(width 0)
-			(type default)
-		)
-	)
-	(wire
-		(pts
 			(xy 121.92 186.69) (xy 125.73 186.69)
 		)
@@
 	(wire
 		(pts
-			(xy 397.51 275.59) (xy 402.59 275.59)
-		)
-		(stroke
-			(width 0)
-			(type default)
-		)
-	)
-	(wire
-		(pts
 			(xy 397.51 248.92) (xy 397.51 254)
 		)
@@
 	(wire
 		(pts
-			(xy 426.72 275.59) (xy 431.8 275.59)
-		)
-		(stroke
-			(width 0)
-			(type default)
-		)
-	)
-	(wire
-		(pts
 			(xy 298.45 191.77) (xy 318.77 191.77)
 		)
@@
 	(wire
 		(pts
+			(xy 34.29 67.31) (xy 52.07 67.31)
+		)
+		(stroke
+			(width 0)
+			(type default)
+		)
+	)
+	(wire
+		(pts
 			(xy 128.27 64.77) (xy 133.35 64.77)
 		)
@@
 	(wire
 		(pts
+			(xy 397.51 265.43) (xy 401.32 265.43)
+		)
+		(stroke
+			(width 0)
+			(type default)
+		)
+	)
+	(wire
+		(pts
 			(xy 121.92 181.61) (xy 121.92 186.69)
 		)
@@
 	(wire
 		(pts
+			(xy 426.72 265.43) (xy 429.26 265.43)
+		)
+		(stroke
+			(width 0)
+			(type default)
+		)
+	)
+	(wire
+		(pts
 			(xy 298.45 176.53) (xy 318.77 176.53)
 		)
@@
 		)
 	)
-	(label "BOOT"
-		(at 402.59 275.59 0)
-		(effects
-			(font
-				(size 1.27 1.27)
-			)
-			(justify left bottom)
-		)
-	)
 	(label "MOSI"
 		(at 297.18 50.8 180)
@@
 		)
 	)
+	(label "BOOT"
+		(at 401.32 265.43 0)
+		(effects
+			(font
+				(size 1.27 1.27)
+			)
+			(justify left bottom)
+		)
+	)
 	(label "MISO"
 		(at 386.08 91.44 180)
@@
 		)
 	)
+	(label "gdo2"
+		(at 34.29 67.31 0)
+		(effects
+			(font
+				(size 1.27 1.27)
+			)
+			(justify left bottom)
+		)
+	)
 	(label "CNS"
 		(at 298.45 204.47 180)
@@
 		)
 	)
+	(label "gdo2"
+		(at 379.73 199.39 0)
+		(effects
+			(font
+				(size 1.27 1.27)
+			)
+			(justify left bottom)
+		)
+	)
 	(label "GDO0"
 		(at 384.81 196.85 0)
@@
 		)
 	)
-	(label "EN"
-		(at 431.8 275.59 0)
-		(effects
-			(font
-				(size 1.27 1.27)
-			)
-			(justify left bottom)
-		)
-	)
 	(label "CE"
 		(at 378.46 86.36 180)
@@
 		(effects
 			(font
+				(size 1.27 1.27)
+			)
+			(justify right bottom)
+		)
+	)
+	(label "EN"
+		(at 429.26 265.43 180)
+		(effects
+			(font

Commit message: changes made the in the header configuration
Parts:
- removed J6: Conn_01x04_Pin, Connector_PinHeader_2.54mm:PinHeader_1x04_P2.54mm_Vertical, symbol Connector:Conn_01x04_Pin
- removed R12, R13: 10K, Resistor_SMD:R_0805_2012Metric, symbol Device:R_Small
- removed SW1: SW_DPST, Button_Switch_SMD:SW_DIP_SPSTx02_Slide_6.7x6.64mm_W6.73mm_P2.54mm_LowProfile_JPin, symbol Switch:SW_DPST
- added D3: D_Zener, Diode_SMD:D_0805_2012Metric, symbol Device:D_Zener
- added J6: Conn_01x05_Pin, Connector_PinHeader_2.54mm:PinHeader_1x05_P2.54mm_Vertical, symbol Connector:Conn_01x05_Pin
- C44: value 10uF -> 22uF
Connections:
- net I0 is gone; now on net GND: U5.16 (I0)
- net I1 is gone; now on net 3v3: U5.17 (I1)
- net IN is gone; now on net Vry: U10.5 (IO5)
- net 3v3: now also J6.1 (Pin_1); no longer D8.1 (K)
- net GND: now also D3.2 (A), J6.2 (Pin_2)
- net GPIO 4: now also U10.11 (IO18); no longer C31.1, U10.4 (IO4)
- net Vin: now also D8.1 (K), D3.1 (K)
- net Vrx: now also U10.4 (IO4), J6.3 (Pin_3); no longer U10.29 (IO36)
- net Vry: now also J6.4 (Pin_4); no longer U10.30 (IO37)
- net at R32.1, U6.3 (Vs): now also C31.1
- net gpio 42: now reaches U10.35 (IO42)
- net gpio 42: now also R33.2
- net gpio 6 renamed SWITCH
- net SWITCH: now also J6.5 (Pin_5); no longer R33.2
Other:
- moved on the sheet: C31, R32, R37
