File: kicad/platy/platy.kicad_pcb (KiCad board)
At the start: 2 copper layers, 125.8 x 52.6 mm, 92 parts, among them J1 Conn_01x04_Socket, J2 Conn_01x02_Socket, J3 Conn_Coaxial, J5 USB_C_Receptacle_USB2.0_16P, J6 Conn_01x05_Pin, J8 Conn_01x14_Socket, J9 Conn_02x04_Odd_Even, Q4 BC847, Q5 Q_PMOS_GSD, SW2 SW_Push(Boot), SW3 SW_Push(EN), U10 ESP32-S3-WROOM-1, U4 CC1101, U5 PN5321A3HN_C1xx, U6 TSOP382xx, U7 AMS1117-3.3, Y2 27.12Mhz, Y3 26MHz

Commit message: added the mounting hole and logo
Parts:
- added REF**: MountingHole_2.2mm_M2_ISO7380, MountingHole:MountingHole_2.2mm_M2_ISO7380, F.Cu at (181.7, 101.5)
- added REF**: MountingHole_2.2mm_M2_ISO7380, MountingHole:MountingHole_2.2mm_M2_ISO7380, F.Cu at (136.8, 101.4)
- added lionckt: LOGO, LOGO, B.Cu at (139.2, 81.6)
Routing:
- net GND: vias 224 -> 221
